File: isopod_distro/isopod_distro.kicad_pcb (KiCad board)
At the start: 4 copper layers, 65 x 56.5 mm, 62 parts, among them J1 CHG_IN, J10 IN 1, J11 IN 2, J12 IN 3, J13 IN 4, J14 IN 5, J15 IN 6, J16 BATT, J17 OUT 7, J18 OUT 8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

Commit message: Add JLC order marking, BOM, gerbs
* Add JLCJLCJLCJLC location for order number
* Add JLC/LCSC BOM database
* Add finished gerbers
Other:
- board text added: "JLCJLCJLCJLC"
